File: fotaoparát_kicad/_autosave-fotaoparát.kicad_pcb (KiCad board)
At the start: 4 copper layers, 22 parts

Commit message: delani pullups
Routing:
- net Net-(ESP32_P4-GPIO39): track 20.7 -> 21.7 mm
Other:
- board text added: "GND"
- board text added: "SW1"
Changed lines of the file:
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@@
 		(net 1)
+	)
+	(gr_text "GND\n"
+		(at 172.5 78.5 0)
+		(layer "F.SilkS")
+		(effects
+			(font
+				(size 1 1)
+				(thickness 0.15)
+			)
+			(justify left bottom)
+		)
+	)
+	(gr_text "SW1"
+		(at 172.5 74.5 0)
+		(layer "F.SilkS")
+		(effects
+			(font
+				(size 1 1)
+				(thickness 0.15)
+			)
+			(justify left bottom)
+		)
 	)
 	(segment
@@
 	)
 	(via
+		(at 170.5 78)
+		(size 3)
+		(drill 1.5)
+		(layers "F.Cu" "B.Cu")
+		(net 1)
+	)
+	(via
 		(at 144 105.5)
 		(size 0.6)
@@
 	(via
 		(at 161.5 101.5)
-		(size 0.6)
-		(drill 0.3)
-		(layers "F.Cu" "B.Cu")
-		(net 1)
-	)
-	(via
-		(at 170.5 73.5)
 		(size 0.6)
 		(drill 0.3)
@@
 	(segment
 		(start 170.5 70)
+		(end 170.5 73.5)
+		(width 0.2)
+		(layer "F.Cu")
+		(net 38)
+	)
+	(segment
+		(start 170.5 70)
 		(end 170.5 70.2525)
 		(width 0.2)
@@
 	)
 	(segment
-		(start 170.5 70)
-		(end 170.5 72.5)
-		(width 0.2)
-		(layer "F.Cu")
-		(net 38)
-	)
-	(segment
 		(start 170.5 67.7475)
 		(end 170.5 70)
@@
 	)
 	(via
-		(at 170.5 72.5)
-		(size 0.6)
-		(drill 0.3)
+		(at 170.5 73.5)
+		(size 3)
+		(drill 1.5)
 		(layers "F.Cu" "B.Cu")
 		(net 38)
