File: fotaoparát_kicad/fotaoparát.kicad_sch (KiCad schematic)
At the start: 46 parts, among them J1 Conn_01x01_Socket, J10 Conn_01x01_Socket, J13 Micro_SD_Card_Det2, J2 Conn_01x01_Socket, J3 Conn_01x01_Socket, J4 Conn_01x01_Socket, J5 Conn_01x01_Socket, J6 Conn_01x01_Socket, J7 Conn_01x01_Socket, J8 Conn_01x01_Socket, J9 Conn_01x01_Socket, SW1 SW_MEC_5G, SW2 SW_MEC_5G

Commit message: vice optimalizace
Changed lines of the file:
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@@
 		(on_board yes)
 		(dnp no)
-		(fields_autoplaced yes)
 		(property "Reference" "#PWR018"
 			(at 314.96 198.12 0)
@@
 		)
 		(property "Value" "GND"
-			(at 314.96 196.85 0)
+			(at 312.42 191.77 0)
 			(effects
 				(font
@@
 		(on_board yes)
 		(dnp no)
-		(fields_autoplaced yes)
 		(property "Reference" "#PWR017"
 			(at 314.96 205.74 0)
@@
 		)
 		(property "Value" "GND"
-			(at 314.96 204.47 0)
+			(at 312.674 199.39 0)
 			(effects
 				(font
@@
 		(on_board yes)
 		(dnp no)
-		(fields_autoplaced yes)
 		(property "Reference" "#PWR011"
 			(at 314.96 213.36 0)
@@
 		)
 		(property "Value" "GND"
-			(at 314.96 212.09 0)
+			(at 312.42 207.01 0)
 			(effects
 				(font
@@
 		(on_board yes)
 		(dnp no)
-		(fields_autoplaced yes)
 		(property "Reference" "#PWR019"
 			(at 314.96 190.5 0)
@@
 		)
 		(property "Value" "GND"
-			(at 314.96 189.23 0)
+			(at 312.166 184.15 0)
 			(effects
 				(font
