File: fotaoparát_kicad/peripherals.kicad_sch (KiCad schematic)
At the start: 27 parts, among them J13 Micro_SD_Card_Det2, J2 BUTTONS

Commit message: Udelal jsem pullupy na tlacitka z fotaku
Parts:
- R8: value 10k -> 330R
- renumbered J2 to J4
Changed lines of the file:
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@@
 		(on_board yes)
 		(dnp no)
-		(property "Reference" "#PWR0101"
+		(property "Reference" "#PWR0104"
 			(at 210.82 29.21 0)
 			(effects
@@
 			(project "fotaoparát"
 				(path "/0ab33720-0b6a-449c-80c0-2b7abe4d9450/be787f52-1025-4e17-92bf-51f58d5e4e6f"
-					(reference "#PWR0101")
+					(reference "#PWR0104")
 					(unit 1)
 				)
@@
 		(dnp no)
 		(fields_autoplaced yes)
-		(property "Reference" "J2"
+		(property "Reference" "J4"
 			(at 261.62 48.2599 0)
 			(effects
@@
 			(project ""
 				(path "/0ab33720-0b6a-449c-80c0-2b7abe4d9450/be787f52-1025-4e17-92bf-51f58d5e4e6f"
-					(reference "J2")
+					(reference "J4")
 					(unit 1)
 				)
@@
 		(on_board yes)
 		(dnp no)
-		(property "Reference" "#PWR0102"
+		(property "Reference" "#PWR0103"
 			(at 210.82 90.17 0)
 			(effects
@@
 			(project "fotaoparát"
 				(path "/0ab33720-0b6a-449c-80c0-2b7abe4d9450/be787f52-1025-4e17-92bf-51f58d5e4e6f"
-					(reference "#PWR0102")
+					(reference "#PWR0103")
 					(unit 1)
 				)
@@
 			)
 		)
-		(property "Value" "10k"
+		(property "Value" "330R"
 			(at 165.862 65.024 90)
 			(effects
