File: fotaoparát_kicad/power.kicad_sch (KiCad schematic)
At the start: 56 parts

Commit message: Zmeny na domacim pc
Other:
- note added: "LENS LOGIC POWER"
- note added: "LENS MAIN POWER"
Changed lines of the file:
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@@
+		)
+	)
+	(text "LENS LOGIC POWER"
+		(exclude_from_sim no)
+		(at 68.58 149.86 0)
+		(effects
+			(font
+				(size 5 5)
+			)
 		)
 	)
@@
 		(effects
 			(font
+				(size 5 5)
+			)
+		)
+	)
+	(text "LENS MAIN POWER"
+		(exclude_from_sim no)
+		(at 185.42 149.86 0)
+		(effects
+			(font
