File: reseni/fotaoparát_kicad/fotaoparát.kicad_pcb (KiCad board)
At the start: 4 copper layers, 102 x 52.8 mm, 120 parts, among them J1 Conn_01x08_Pin, J13 Micro_SD_Card_Det2, J2 Conn_01x01_Socket, J3 Conn_01x01_Socket, J4 BUTTONS, J5 Conn_01x01_Socket, SW1 SW_MEC_5G, SW2 SW_MEC_5G, U1 TLV62569DBV, Y2 Crystal_GND24

Commit message: je to bordel, snad bude ale fungovat
Parts:
- removed BAT_IN1, BAT_OUT1: Conn_01x01_Socket, Connector_Wire:SolderWirePad_1x01_SMD_1.5x3mm
- removed the R8 at (145.6, 101.5)
- removed the R8 at (190.4, 130.0)
- removed Y2: Crystal_GND24, Crystal:Crystal_SMD_Abracon_ABM8G-4Pin_3.2x2.5mm
- removed svviit_design: LOGO, LOGO
- added BAT_IO1: Conn_01x02_Socket, Connector_Wire:SolderWire-1.5sqmm_1x02_P6mm_D1.7mm_OD3mm, F.Cu at (59.9, 159.7)
- added C59: 12pF, Capacitor_SMD:C_0402_1005Metric, F.Cu at (273.2, 103.6)
- added C63: 12pF, Capacitor_SMD:C_0402_1005Metric, F.Cu at (273.2, 105.6)
- added C64: 10uF, Capacitor_SMD:C_0603_1608Metric, B.Cu at (144.5, 103.2)
- added R14: 4k7, Resistor_SMD:R_0603_1608Metric, F.Cu at (265.1, 78.1)
- added R27: 22R, Resistor_SMD:R_0402_1005Metric, F.Cu at (141.3, 100.2)
- added R8: 10k, Resistor_SMD:R_0603_1608Metric, F.Cu at (261.1, 83.1)
- added Y1: 40MHz +/- 10ppm 10pF, Crystal:Crystal_SMD_2016-4Pin_2.0x1.6mm, F.Cu at (142.0, 97.4)
- C1, C11, C12, C13, C15, C2, C21, C42, J1, J4, LOGIC_CONVERT1, R10, R11, R12: moved to F.Cu
- C23, CAM_IN1, DISPLAY_IN1: moved to B.Cu
- C24, C35, C36, C38, C39: value 100nF -> 10uF; footprint Capacitor_SMD:C_0201_0603Metric -> Capacitor_SMD:C_0603_1608Metric
- C25: value 1uF -> 10uF; footprint Capacitor_SMD:C_0201_0603Metric -> Capacitor_SMD:C_0603_1608Metric; moved to B.Cu
- C26: value 1uF -> 10nF; moved to B.Cu
- C3, C30, C34: footprint Capacitor_SMD:C_0201_0603Metric -> Capacitor_SMD:C_0603_1608Metric
- C31, C32: value 100nF -> 1uF
- C33: value 10uF -> 1uF
- C37, C40: value 10pF -> 10uF; footprint Capacitor_SMD:C_0201_0603Metric -> Capacitor_SMD:C_0603_1608Metric; moved to B.Cu
- C43, C45, C48, C50, C6, C8: footprint Capacitor_SMD:C_0603_1608Metric -> Capacitor_SMD:C_0201_0603Metric
- ESP32_P4: footprint PCM_Espressif:ESP32-P4 -> Espressif:ESP32-P4
- ESP_FLASH1: footprint PCM_SamacSys_Parts:SON127P800X600X80-9N-D -> SamacSys_Parts:SON127P800X600X80-9N-D
- moved SW1 154.4 mm to (270.5, 87.2), turned to 0 degrees
- moved C13 153.6 mm to (265.7, 104.0), turned to 0 degrees
- moved SW2 149.3 mm to (270.5, 91.8), turned to 0 degrees
- moved R12 149.0 mm to (261.1, 90.6)
- moved C11 144.5 mm to (265.7, 100.5), turned to 0 degrees
- moved R11 140.8 mm to (261.1, 88.1), turned to 0 degrees
- moved C21 129.2 mm to (268.1, 104.0)
- moved D4 125.8 mm to (63.4, 166.9)
- moved C10 124.8 mm to (59.1, 168.6), turned to 0 degrees
- moved L1 123.6 mm to (59.1, 171.1)
- moved C9 122.1 mm to (59.1, 166.1), turned to 0 degrees
- moved C8 121.9 mm to (62.4, 171.0), turned to 0 degrees
- moved D1 121.0 mm to (63.4, 163.8), turned to 0 degrees
- moved R10 119.5 mm to (261.1, 85.6), turned to 0 degrees
- moved C7 118.8 mm to (59.1, 163.5)
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Connections:
- net Net-(ESP32_P4-EN_DCDC) renamed /EN_DCDC
- C11 pad 1: Net-(ESP32_P4-CHIP_PU) -> GND
- C11 pad 2: GND -> Net-(ESP32_P4-CHIP_PU)
- C13 pad 2: unconnected-(C13-Pad2) -> GND
- C15 pad 1: /ESP_VDD_HP -> +1V1
- C18 pad 1: +3V3 -> GND
- C18 pad 2: GND -> +3V3
- C19 pad 1: +3V3 -> GND
- C19 pad 2: GND -> +3V3
- C20 pad 1: /ESP_VDD_HP -> +3V3
- C21 pad 1: /ESP_VDD_HP -> GND
- C21 pad 2: GND -> +1V1
- C22 pad 1: /ESP_VDD_HP -> +1V1
- C23 pad 1: +3V3 -> GND
- C23 pad 2: GND -> +1V1
- C24 pad 1: +3V3 -> GND
- C24 pad 2: GND -> +3V3
- C25 pad 1: /VDDO_FLASH -> GND
- C25 pad 2: GND -> +3V3
- C26 pad 1: /VDDO_PSRAM -> /VDDO_3
- C27 pad 1: +3V3 -> /VDDO_3
- C31 pad 1: /VDD_PSRAM_0 -> /VDDO_FLASH
- C32 pad 1: /VDD_PSRAM_1 -> /VDDO_PSRAM
- C33 pad 1: +3V3 -> /VDDO_3
- C34 pad 1: /VDDO_3 -> GND
- C34 pad 2: GND -> +3V3
- C35 pad 1: +3V3 -> GND
- C35 pad 2: GND -> +3V3
- C36 pad 1: +3V3 -> GND
- C36 pad 2: GND -> +3V3
- C37 pad 2: Net-(ESP32_P4-XTAL_P) -> +3V3
- C38 pad 1: +3V3 -> GND
- C38 pad 2: GND -> +3V3
- C39 pad 1: /VDDO_3 -> GND
- C39 pad 2: GND -> +1V1
- C40 pad 1: Net-(ESP32_P4-XTAL_N) -> GND
- C40 pad 2: GND -> +1V1
- C42 pad 1: /ESP_VDD_HP -> +1V1
- ESP32_P4 pad 100: Net-(ESP32_P4-XTAL_P) -> /XTAL_P
- ESP32_P4 pad 26: /ESP_VDD_HP -> +1V1
- ESP32_P4 pad 49: /USB_DATA_N -> USB_DATA_N
- ESP32_P4 pad 50: /USB_DATA_P -> USB_DATA_P
- ESP32_P4 pad 76: /ESP_VDD_HP -> +1V1
- ESP32_P4 pad 78: unconnected-(ESP32_P4-FB_DCDC-Pad78) -> /FB_DCDC
- ESP32_P4 pad 91: /ESP_VDD_HP -> +1V1
- ESP32_P4 pad 99: Net-(ESP32_P4-XTAL_N) -> /XTAL_N
- L2 pad 2: /ESP_VDD_HP -> +1V1
- R25 pad 1: /ESP_VDD_HP -> +1V1
- R25 pad 2: Net-(U1-FB) -> /FB_DCDC
- R26 pad 1: Net-(U1-FB) -> /FB_DCDC
- SW1 pad 2: GND -> Net-(ESP32_P4-GPIO35)
- U1 pad 5: Net-(U1-FB) -> /FB_DCDC
Routing:
- net GND: track 195.5 -> 54.5 mm, vias 49 -> 10
- net LED_A: track 99.8 -> 0.00 mm, vias 2 -> 0
- net +7V2: track 95.5 -> 0.00 mm, vias 2 -> 0
- net BUTT_4: track 90.5 -> 0.00 mm, vias 2 -> 0
- net BUTT_2: track 90.0 -> 0.00 mm, vias 2 -> 0
- net BUTT_5: track 89.8 -> 0.00 mm, vias 2 -> 0
- net BUTT_3: track 89.7 -> 0.00 mm, vias 2 -> 0
- net BUTT_1: track 89.3 -> 0.00 mm, vias 2 -> 0
- net BUTT_6: track 88.9 -> 0.00 mm, vias 2 -> 0
- net BUTT_8: track 88.6 -> 0.00 mm, vias 2 -> 0
- net BUTT_7: track 88.4 -> 0.00 mm, vias 2 -> 0
- net +5V5: track 88.1 -> 0.00 mm, vias 3 -> 0
- net BUTT_9: track 88.0 -> 0.00 mm, vias 2 -> 0
- net USB_DATA_N: track 76.3 -> 0.00 mm, vias 3 -> 0
- net Net-(ESP32_P4-GPIO27/ADC/USB): track 73.7 -> 0.00 mm, vias 2 -> 0
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