File: reseni/fotaoparát_kicad/fotaoparát.kicad_sch (KiCad schematic)
At the start: 36 parts, among them J1 Conn_01x08_Pin, J2 Conn_01x01_Socket, J3 Conn_01x01_Socket, J5 Conn_01x01_Socket, SW1 SW_MEC_5G, SW2 SW_MEC_5G, U1 TLV62569DBV, Y1 40MHz +/- 10ppm 10pF

Commit message: je to bordel, snad bude ale fungovat
Parts:
- added C16, C17, C18, C19, C20, C21, C22, C23, C27: 100nF, Capacitor_SMD:C_0201_0603Metric, symbol Device:C
- added C24, C25, C34, C35, C36, C37, C38, C39, C40, C64: 10uF, Capacitor_SMD:C_0603_1608Metric, symbol Device:C
- added C26: 10nF, Capacitor_SMD:C_0201_0603Metric, symbol Device:C
- added C28, C31, C32, C33: 1uF, Capacitor_SMD:C_0201_0603Metric, symbol Device:C
- C12: LSCS Number C307385 -> C668346
- C15, C42: LCSC Part (none) -> C59461
- ESP32_P4: footprint PCM_Espressif:ESP32-P4 -> Espressif:ESP32-P4
- ESP_FLASH1: footprint PCM_SamacSys_Parts:SON127P800X600X80-9N-D -> SamacSys_Parts:SON127P800X600X80-9N-D
- R27: value 22 -> 22R; LSCS Number (none) -> C25092
Connections:
- net +3V3: now also C16.1, C17.1, C18.2, C19.2, C20.1, C24.2, C25.2, C34.2, C35.2, C36.2, C37.2, C38.2
- net GND: now also C16.2, C17.2, C18.1, C19.1, C20.2, C21.1, C22.2, C23.1, C24.1, C25.1, C26.2, C27.2, C28.2, C31.2, C32.2, C33.2, C34.1, C35.1, C36.1, C37.1, C38.1, C39.1, C40.1, C64.1
- net VDDO_3: now also C26.1, C27.1, C28.1, C33.1
- net VDDO_FLASH: now also C31.1
- net VDDO_PSRAM: now also C32.1
- net ESP_VDD_HP renamed +1V1
- net +1V1: now also C21.2, C22.1, C23.2, C39.2, C40.2, C64.2
Other:
- sheet POWER ports: added none; removed VDDO_3, VDDO_FLASH, VDDO_PSRAM, VDD_ANA, VDD_BAT, VDD_DCDCC, VDD_FLASHIO, VDD_HP_0, VDD_HP_2, VDD_HP_3, VDD_IO_0, VDD_IO_4, VDD_IO_5, VDD_IO_6, VDD_LDO, VDD_LP, VDD_PSRAM_0, VDD_PSRAM_1, VDD_USBPHY
- note added: "Entry point decoupling"
- note added: "FLASH BTN"
- note added: "Na vývodech!"
- note added: "VDD_HP_0"
- note added: "VDD_HP_2"
- note added: "VDD_HP_3"
- note added: "VDD_IO_0"
- note added: "VDD_IO_4"
- note added: "VDD_IO_5"
- note added: "VDD_IO_6"
- note added: "VDD_LP"
- moved on the sheet: C1, C12, C2, ESP_FLASH1, R13, R14
