File: reseni/fotaoparát_kicad/peripherals.kicad_sch (KiCad schematic)
At the start: 27 parts, among them J13 Micro_SD_Card_Det2, J4 BUTTONS

Commit message: je to bordel, snad bude ale fungovat
Parts:
- C3, C30: footprint Capacitor_SMD:C_0201_0603Metric -> Capacitor_SMD:C_0603_1608Metric
Changed lines of the file:
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@@
 			)
 		)
-		(property "Footprint" "Capacitor_SMD:C_0201_0603Metric"
+		(property "Footprint" "Capacitor_SMD:C_0603_1608Metric"
 			(at 54.61 25.7048 0)
 			(hide yes)
@@
 			)
 		)
-		(property "Footprint" "Capacitor_SMD:C_0201_0603Metric"
+		(property "Footprint" "Capacitor_SMD:C_0603_1608Metric"
 			(at 134.62 24.4348 0)
 			(hide yes)
