File: reseni/fotaoparát_kicad/power.kicad_sch (KiCad schematic)
At the start: 56 parts

Commit message: je to bordel, snad bude ale fungovat
Parts:
- removed C16, C17, C18, C19, C20, C21, C22, C23, C24, C27, C31, C32, C35, C36, C38, C39: 100nF, Capacitor_SMD:C_0201_0603Metric, symbol Device:C
- removed C25, C26, C28: 1uF, Capacitor_SMD:C_0201_0603Metric, symbol Device:C
- removed C33, C34: 10uF, Capacitor_SMD:C_0201_0603Metric, symbol Device:C
- C43, C45, C48, C50, C6, C8: footprint Capacitor_SMD:C_0603_1608Metric -> Capacitor_SMD:C_0201_0603Metric; LSCS Number C66501 -> C668346
Other:
- note removed: "ANALOG POWER PINS"
- note removed: "CAPACITORS MEANT TO BE PLACED DIRECTLY ON THE PIN"
- note removed: "DIGITAL CORE POWER PINS"
- note removed: "FLASH/PSRAM IO POWER PINS"
- note removed: "HP/LP POWER PINS"
- note removed: "INTERNAL LDO/DCDC OUPUT PINS"
- note removed: "LDO OUTPUT PINS"
- note removed: "MIPI PHY POWER"
- note removed: "USB PHY POWER"
- moved on the sheet: ESD_PROT1, R1, R9, USB-C_2.0
